Commit message: Integrate approved Silverhand rover model

File: silverhand_rover_description/ros2_control/silverhand_rover.ros2_control.xacro (robot description, xacro)
@@ -22,43 +22,43 @@
         </xacro:unless>
       </hardware>
-      <joint name="front_left_wheel_joint">
+      <joint name="left_front_wheel_joint">
         <command_interface name="velocity"/>
         <state_interface name="position">
-          <param name="initial_value">${initial_positions['front_left_wheel_joint']}</param>
+          <param name="initial_value">${initial_positions['left_front_wheel_joint']}</param>
         </state_interface>
         <state_interface name="velocity"/>
       </joint>
-      <joint name="middle_left_wheel_joint">
+      <joint name="left_middle_wheel_joint">
         <command_interface name="velocity"/>
         <state_interface name="position">
-          <param name="initial_value">${initial_positions['middle_left_wheel_joint']}</param>
+          <param name="initial_value">${initial_positions['left_middle_wheel_joint']}</param>
         </state_interface>
         <state_interface name="velocity"/>
       </joint>
-      <joint name="rear_left_wheel_joint">
+      <joint name="left_rear_wheel_joint">
         <command_interface name="velocity"/>
         <state_interface name="position">
-          <param name="initial_value">${initial_positions['rear_left_wheel_joint']}</param>
+          <param name="initial_value">${initial_positions['left_rear_wheel_joint']}</param>
         </state_interface>
         <state_interface name="velocity"/>
       </joint>
-      <joint name="front_right_wheel_joint">
+      <joint name="right_front_wheel_joint">
         <command_interface name="velocity"/>
         <state_interface name="position">
-          <param name="initial_value">${initial_positions['front_right_wheel_joint']}</param>
+          <param name="initial_value">${initial_positions['right_front_wheel_joint']}</param>
         </state_interface>
         <state_interface name="velocity"/>
       </joint>
-      <joint name="middle_right_wheel_joint">
+      <joint name="right_middle_wheel_joint">
         <command_interface name="velocity"/>
         <state_interface name="position">
-          <param name="initial_value">${initial_positions['middle_right_wheel_joint']}</param>
+          <param name="initial_value">${initial_positions['right_middle_wheel_joint']}</param>
         </state_interface>
         <state_interface name="velocity"/>
       </joint>
-      <joint name="rear_right_wheel_joint">
+      <joint name="right_rear_wheel_joint">
         <command_interface name="velocity"/>
         <state_interface name="position">
-          <param name="initial_value">${initial_positions['rear_right_wheel_joint']}</param>
+          <param name="initial_value">${initial_positions['right_rear_wheel_joint']}</param>
         </state_interface>
         <state_interface name="velocity"/>

File: silverhand_rover_description/urdf/silverhand_rover.urdf.xacro (robot description, xacro)
@@ -8,7 +8,6 @@
   <xacro:arg name="node_id" default="110"/>
   <xacro:arg name="queue_len" default="1000"/>
-  <xacro:include filename="$(find silverhand_rover_description)/urdf/silverhand_rover.urdf"/>
-  <xacro:include
-    filename="$(find silverhand_rover_description)/ros2_control/silverhand_rover.ros2_control.xacro"/>
+  <xacro:include filename="$(find silverhand_rover_description)/urdf/silverhand_rover_model.urdf.xacro"/>
+  <xacro:include filename="$(find silverhand_rover_description)/ros2_control/silverhand_rover.ros2_control.xacro"/>
   <xacro:silverhand_rover_ros2_control
     name="SilverhandRoverSystem"
